File: HW/Solar_Array/Solar_Array.kicad_pcb (KiCad board)
At the start: 2 copper layers, 40 x 40 mm, 36 parts, among them J1 Conn_01x02, J3 Conn_01x02, J8 Conn_01x02, J9 Conn_01x02

Commit message: start
Parts:
- D21, D22, D23, D24, D25, D26, D27, D28, D29, D30, D31, D32, D33, D34, D35, D36: footprint OptoDevice:Osram_DIL2_4.3x4.65mm_P5.08mm -> solarzellen:Osram_DIL2_4.3x4.65mm_P5.08mm
