File: HW/Solar_Array/Solar_Array.kicad_sch (KiCad schematic)
At the start: 36 parts, among them J1 Conn_01x02, J2 Conn_01x02, J3 Conn_01x02, J4 Conn_01x02

Commit message: start
Changed lines of the file:
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@@
 (kicad_sch
-	(version 20231120)
+	(version 20250114)
 	(generator "eeschema")
-	(generator_version "8.0")
+	(generator_version "9.0")
 	(paper "A4")
+	(rectangle
+		(start 233.68 72.39)
+		(end 261.62 121.92)
+		(stroke
+			(width 1)
+			(type dash)
+			(color 255 0 255 0.6)
+		)
+		(fill
+			(type none)
+		)
+	)
+	(rectangle
+		(start 50.8 54.61)
+		(end 88.9 139.7)
+		(stroke
+			(width 1)
+			(type dash)
+			(color 0 255 255 0.5)
+		)
+		(fill
+			(type none)
+		)
+	)
+	(rectangle
+		(start 114.3 54.61)
+		(end 205.74 139.7)
+		(stroke
+			(width 1)
+			(type dash)
+			(color 0 255 255 0.5)
+		)
+		(fill
+			(type none)
+		)
+	)
+	(text "Solar Array\n"
+		(exclude_from_sim no)
+		(at 160.528 51.816 0)
+		(effects
+			(font
+				(size 2 2)
+			)
+		)
+	)
+	(text "Storage"
+		(exclude_from_sim no)
+		(at 69.85 51.816 0)
+		(effects
+			(font
+				(size 2 2)
+			)
+		)
+	)
+	(text "Headers"
+		(exclude_from_sim no)
+		(at 247.142 70.104 0)
+		(effects
+			(font
+				(size 2 2)
+			)
+		)
+	)
 	(junction
 		(at 179.07 128.27)
@@
 		)
 	)
-	(rectangle
-		(start 233.68 72.39)
-		(end 261.62 121.92)
-		(stroke
-			(width 1)
-			(type dash)
-			(color 255 0 255 0.6)
-		)
-		(fill
-			(type none)
-		)
-	)
-	(rectangle
-		(start 50.8 54.61)
-		(end 88.9 139.7)
-		(stroke
-			(width 1)
-			(type dash)
-			(color 0 255 255 0.5)
-		)
-		(fill
-			(type none)
-		)
-	)
-	(rectangle
-		(start 114.3 54.61)
-		(end 205.74 139.7)
-		(stroke
-			(width 1)
-			(type dash)
-			(color 0 255 255 0.5)
-		)
-		(fill
-			(type none)
-		)
-	)
-	(text "Solar Array\n"
-		(exclude_from_sim no)
-		(at 160.528 51.816 0)
-		(effects
-			(font
-				(size 2 2)
-			)
-		)
-	)
-	(text "Storage"
-		(exclude_from_sim no)
-		(at 69.85 51.816 0)
-		(effects
-			(font
-				(size 2 2)
-			)
-		)
-	)
-	(text "Headers"
-		(exclude_from_sim no)
-		(at 247.142 70.104 0)
-		(effects
-			(font
-				(size 2 2)
-			)
-		)
-	)
 	(label "+PD"
 		(at 69.85 63.5 0)
@@
 		)
 	)
+	(embedded_fonts no)
 )
